File: Hardware/schematics/kicad/craig-andreas-8ch-midi-to-cv.kicad_pcb (KiCad board)
At the start: 2 copper layers, 99.8 x 108.5 mm, 194 parts, among them J1 MIDI IN, J10 Osc CV Out 2, J11 Velocity CV Out, J12 Filter CV Out, J13 Bend/Mod CV Out, J14 Gate Out, J15 Trig Out, J16 SSD1306, J2 USB_A, J3 Eurorack Power 16 pin, J4 Saw-In-2, J5 Saw-In-1, J6 LFO_RATE, J7 LFO_WAVE, J8 Panel Buttons, J9 Osc CV Out 1, U1 Teensy4.1, U10 DAC8568, U12 Electric Druid TAPLFO 3, U13 AS3360, U14 L7905, U15 74HC595, U16 74HC595, U17 74HC595, U18 LM2902, U19 LM2902, U2 DAC8568, U20 LM2902, U21 LM2902, U22 LM2902, U23 LM2902, U24 LM2902, U25 LM2902, U26 LM2902, U27 74HC165, U3 ADG5206BRUZ, U4 74HC14, U5 TL074HID, U7 DAC8568, U8 DAC8568, U9 DAC8568

Commit message: Remove LFO in favor of standalone LFO and create PCB. FM Input still exists in case it's needed.
Parts:
- removed C17, C18, C19, C20, C22, C24, C25, C26, C28, C8: 100nF, Capacitor_SMD:C_0805_2012Metric_Pad1.18x1.45mm_HandSolder
- removed C35, C37: 10nF, Capacitor_SMD:C_0805_2012Metric_Pad1.18x1.45mm_HandSolder
- removed C36, C38: 2.2nF, Capacitor_SMD:C_0805_2012Metric_Pad1.18x1.45mm_HandSolder
- removed C39: 560pF, Capacitor_SMD:C_0805_2012Metric_Pad1.18x1.45mm_HandSolder
- removed D3: LED, Eurocad:LED3mm
- removed D4, D5: BAT43WS, Diode_SMD:D_SOD-323_HandSoldering
- removed J6: LFO_RATE, Connector_Wire:SolderWirePad_1x01_SMD_2x4mm
- removed J7: LFO_WAVE, Connector_Wire:SolderWirePad_1x01_SMD_2x4mm
- removed R10, R11, R4, R5: 10k, PCM_Resistor_SMD_AKL:R_0805_2012Metric_Pad1.15x1.40mm_HandSolder
- removed R12: 24k, PCM_Resistor_SMD_AKL:R_0805_2012Metric_Pad1.15x1.40mm_HandSolder
- removed R13, R14, R15, R8: 47k, PCM_Resistor_SMD_AKL:R_0805_2012Metric_Pad1.15x1.40mm_HandSolder
- removed R16: 1k, PCM_Resistor_SMD_AKL:R_0805_2012Metric_Pad1.15x1.40mm_HandSolder
- removed R6: 220, PCM_Resistor_SMD_AKL:R_0805_2012Metric_Pad1.15x1.40mm_HandSolder
- removed R7, R9: 12k, PCM_Resistor_SMD_AKL:R_0805_2012Metric_Pad1.15x1.40mm_HandSolder
- removed RV2: Offset 100k, PCM_Potentiometer_THT_AKL:Potentiometer_Runtron_RM-065_Vertical
- removed RV3: 100k, PCM_Potentiometer_THT_AKL:Potentiometer_Runtron_RM-065_Vertical
- removed RV4: 100k set 1.65v, Pot-User:Potentiometer_Bourns_3296W_Vertical-User
- removed U12: Electric Druid TAPLFO 3, PCM_Package_DIP_AKL:DIP-14_W7.62mm_LongPads
- removed U13: AS3360, Package_DIP:DIP-14_W7.62mm_LongPads
- removed U14: L7905, PCM_4ms_Package_TO:TO-220-3_Vertical
- removed U5: TL074HID, PCM_Package_SO_AKL:SOIC-14_3.9x8.7mm_P1.27mm
- added J17: USB Teensy, Connector_JST:JST_XH_B2B-XH-A_1x02_P2.50mm_Vertical, F.Cu at (88.7, 63.6)
- added REF**: MountingHole_2.2mm_M2_ISO7380, MountingHole:MountingHole_2.2mm_M2_ISO7380, F.Cu at (147.3, 151.2)
- added REF**: MountingHole_2.2mm_M2_ISO7380, MountingHole:MountingHole_2.2mm_M2_ISO7380, F.Cu at (53.5, 48.7)
- added REF**: MountingHole_2.2mm_M2_ISO7380, MountingHole:MountingHole_2.2mm_M2_ISO7380, F.Cu at (53.5, 151.2)
- added REF**: MountingHole_2.2mm_M2_ISO7380, MountingHole:MountingHole_2.2mm_M2_ISO7380, F.Cu at (147.3, 48.7)
- C1, C11, C16, C2, C21, C23, C27, C29, C3, C30, C31, C4, C5, C7, D1, J3, R1, R2, R33, R34, R37, R38, R39, R40, R43, R44, R45, R46, R49, R50, R51, R52, R53, R54, R57, R58, R61, R62, R67, R68, R71, R72, R75, R76, R77, R79, R80, R81, R82, R85, R86, R89, R90, R93, R94, U1, U10, U18, U2, U20, U22, U24, U26, U27, U7, U8, U9: moved to B.Cu
- J10, J11, J9: footprint Connector_JST:JST_XH_B9B-XH-A_1x09_P2.50mm_Vertical -> Connector_IDC:IDC-Header_2x05_P2.54mm_Vertical
- RV1: footprint PCM_Potentiometer_THT_AKL:Potentiometer_Runtron_RM-065_Vertical -> Potentiometer_THT:Potentiometer_Runtron_RM-065_Vertical; moved to B.Cu
- U4: footprint Package_DIP:DIP-14_W7.62mm_LongPads -> Package_SO:SOIC-14_3.9x8.7mm_P1.27mm
- moved U26 173.6 mm to (107.7, 118.9), turned to 90 degrees
- moved U20 161.9 mm to (120.0, 101.5), turned to 90 degrees
- moved U23 160.9 mm to (122.4, 120.0), turned to 90 degrees
- moved U19 153.3 mm to (118.7, 89.4), turned to 90 degrees
- moved R95 152.1 mm to (113.5, 115.0), turned to 180 degrees
- moved RV1 151.3 mm to (67.4, 82.7)
- moved R104 150.4 mm to (56.9, 109.7), turned to 90 degrees
- moved R89 149.9 mm to (127.9, 122.3)
- moved R88 149.4 mm to (126.0, 115.0), turned to 180 degrees
- moved R91 149.1 mm to (128.2, 127.1), turned to -90 degrees
- moved R96 148.5 mm to (116.8, 116.6), turned to -90 degrees
- moved R105 148.4 mm to (59.4, 109.7), turned to 90 degrees
- moved R93 148.1 mm to (119.3, 113.3), turned to 90 degrees
- moved U22 148.0 mm to (126.4, 116.7), turned to 180 degrees
- moved J16 147.8 mm to (70.3, 87.9)
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Connections:
- C12 pad 1: GND -> +3.3V
- C12 pad 2: -12V -> GND
- C13 pad 1: GND -> +3.3V
- C13 pad 2: -12V -> GND
- C14 pad 1: GND -> +3.3V
- C14 pad 2: -12V -> GND
- C15 pad 1: +12V -> +3.3V
- C16 pad 1: GND -> +5V
- C16 pad 2: -12V -> GND
- C21 pad 1: +12V -> +5V
- C9 pad 1: +12V -> +3.3V
- R35 pad 1: Net-(U18B--) -> Net-(U19C--)
- R36 pad 2: Net-(U18B--) -> Net-(U19C--)
- R39 pad 1: Net-(U18D--) -> Net-(U19A--)
- R40 pad 2: Net-(U18D--) -> Net-(U19A--)
- R41 pad 1: Net-(U19A--) -> Net-(U18D--)
- R42 pad 2: Net-(U19A--) -> Net-(U18D--)
- R45 pad 1: Net-(U19C--) -> Net-(U18B--)
- R46 pad 2: Net-(U19C--) -> Net-(U18B--)
- R51 pad 1: Net-(U20B--) -> Net-(U21A--)
- R52 pad 2: Net-(U20B--) -> Net-(U21A--)
- R55 pad 1: Net-(U20D--) -> Net-(U21C--)
- R56 pad 2: Net-(U20D--) -> Net-(U21C--)
- R57 pad 1: Net-(U21A--) -> Net-(U20B--)
- R58 pad 2: Net-(U21A--) -> Net-(U20B--)
- R61 pad 1: Net-(U21C--) -> Net-(U20D--)
- R62 pad 2: Net-(U21C--) -> Net-(U20D--)
- R67 pad 1: Net-(U25C--) -> Net-(U24D--)
- R68 pad 2: Net-(U25C--) -> Net-(U24D--)
- R71 pad 1: Net-(U25A--) -> Net-(U24B--)
- R72 pad 2: Net-(U25A--) -> Net-(U24B--)
- R73 pad 1: Net-(U24D--) -> Net-(U25C--)
- R74 pad 2: Net-(U24D--) -> Net-(U25C--)
- R77 pad 1: Net-(U24B--) -> Net-(U25A--)
- R78 pad 2: Net-(U24B--) -> Net-(U25A--)
- R83 pad 1: Net-(U22B--) -> Net-(U23A--)
- R84 pad 2: Net-(U22B--) -> Net-(U23A--)
- R87 pad 1: Net-(U22D--) -> Net-(U23C--)
- R88 pad 2: Net-(U22D--) -> Net-(U23C--)
- R89 pad 1: Net-(U23A--) -> Net-(U22B--)
- R90 pad 2: Net-(U23A--) -> Net-(U22B--)
- R93 pad 1: Net-(U23C--) -> Net-(U22D--)
- R94 pad 2: Net-(U23C--) -> Net-(U22D--)
- U1 pad 66: unconnected-(U1-D--Pad66) -> Net-(J17-Pin_1)
- U1 pad 67: unconnected-(U1-D+-Pad67) -> Net-(J17-Pin_2)
- U18 pad 12: DAC_CV4 -> DAC_CV5
- U18 pad 14: Net-(J9-Pin_4) -> Net-(J9-Pin_5)
- U18 pad 5: DAC_CV2 -> DAC_CV7
- U18 pad 7: Net-(J9-Pin_2) -> Net-(J9-Pin_7)
- U19 pad 1: Net-(J9-Pin_5) -> Net-(J9-Pin_4)
- U19 pad 10: DAC_CV7 -> DAC_CV2
- U19 pad 3: DAC_CV5 -> DAC_CV4
- U19 pad 8: Net-(J9-Pin_7) -> Net-(J9-Pin_2)
- U20 pad 12: DAC_CV12 -> DAC_CV15
- U20 pad 14: Net-(J10-Pin_4) -> Net-(J10-Pin_7)
- U20 pad 5: DAC_CV10 -> DAC_CV13
- U20 pad 7: Net-(J10-Pin_2) -> Net-(J10-Pin_5)
- U21 pad 1: Net-(J10-Pin_5) -> Net-(J10-Pin_2)
- U21 pad 10: DAC_CV15 -> DAC_CV12
- U21 pad 3: DAC_CV13 -> DAC_CV10
- U21 pad 8: Net-(J10-Pin_7) -> Net-(J10-Pin_4)
- U22 pad 12: DAC_VEL4 -> DAC_VEL7
- U22 pad 14: Net-(J11-Pin_4) -> Net-(J11-Pin_7)
- U22 pad 5: DAC_VEL2 -> DAC_VEL5
- U22 pad 7: Net-(J11-Pin_2) -> Net-(J11-Pin_5)
- U23 pad 1: Net-(J11-Pin_5) -> Net-(J11-Pin_2)
- U23 pad 10: DAC_VEL7 -> DAC_VEL4
- U23 pad 3: DAC_VEL5 -> DAC_VEL2
- U23 pad 8: Net-(J11-Pin_7) -> Net-(J11-Pin_4)
- U24 pad 12: DAC_FCV4 -> DAC_FCV7
- U24 pad 14: Net-(J12-Pin_4) -> Net-(J12-Pin_7)
- U24 pad 5: DAC_FCV2 -> DAC_FCV5
- U24 pad 7: Net-(J12-Pin_2) -> Net-(J12-Pin_5)
- U25 pad 1: Net-(J12-Pin_5) -> Net-(J12-Pin_2)
- U25 pad 10: DAC_FCV7 -> DAC_FCV4
- U25 pad 3: DAC_FCV5 -> DAC_FCV2
- U25 pad 8: Net-(J12-Pin_7) -> Net-(J12-Pin_4)
Routing:
- net +5V: track 0.00 -> 307.4 mm, vias 0 -> 7
- net +12V: track 0.00 -> 278.0 mm, vias 0 -> 5
- net +3.3V: track 0.00 -> 204.0 mm, vias 0 -> 8
- net GND: track 0.00 -> 158.0 mm, vias 0 -> 457
- net DAC_SCL: track 0.00 -> 73.1 mm, vias 0 -> 5
- net DAC_SDA: track 0.00 -> 58.5 mm, vias 0 -> 5
- net Net-(U3-D): track 0.00 -> 55.0 mm, vias 0 -> 2
- net DAC_VEL5: track 0.00 -> 44.6 mm
- net Net-(J11-Pin_2): track 0.00 -> 43.3 mm
- net DAC_VEL1: track 0.00 -> 43.3 mm, vias 0 -> 2
- net Net-(J10-Pin_3): track 0.00 -> 40.0 mm, vias 0 -> 1
- net Net-(J10-Pin_2): track 0.00 -> 39.8 mm, vias 0 -> 3
- net Net-(J10-Pin_8): track 0.00 -> 39.6 mm, vias 0 -> 2
- net -12V: track 0.00 -> 35.9 mm, vias 0 -> 1
- net DAC_VEL3: track 0.00 -> 34.8 mm
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Other:
- board text added: "D+"
- board text added: "D-"
